File: AquariumSensor.kicad_sch (KiCad schematic)
At the start: 13 parts, among them J1 Conn_YF_S201, J2 Conn_KS0429, J3 Barrel_Jack, SW1 SW_Reed, SW2 SW_Reed, U1 WeMos_D1_mini, U2 DS18B20, U3 DHT11, U4 AM312_breakout

Commit message: 1.1 Release to fix wrong polarity on J3 DC Jack
Connections:
- net at J1.1 (VCC), J2.2 (VIN), U1.9 (5V)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: now also J3.1; no longer J3.2
- net at J1.2 (GND), J2.3 (GND), SW1.1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: now also J3.2; no longer J3.1
Other:
- moved on the sheet: J3
Changed lines of the file:
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@@
+	)
+	(junction
+		(at 74.93 73.66)
+		(diameter 0)
+		(color 0 0 0 0)
+	)
+	(junction
+		(at 102.87 127)
+		(diameter 0)
+		(color 0 0 0 0)
+	)
+	(junction
+		(at 105.41 82.55)
+		(diameter 0)
+		(color 0 0 0 0)
 	)
 	(junction
@@
 	)
 	(junction
-		(at 74.93 73.66)
-		(diameter 0)
-		(color 0 0 0 0)
-	)
-	(junction
-		(at 26.67 76.2)
-		(diameter 0)
-		(color 0 0 0 0)
-	)
-	(junction
-		(at 102.87 127)
-		(diameter 0)
-		(color 0 0 0 0)
-	)
-	(junction
-		(at 105.41 82.55)
-		(diameter 0)
-		(color 0 0 0 0)
-	)
-	(junction
 		(at 36.83 76.2)
 		(diameter 0)
@@
 	)
 	(junction
+		(at 26.67 125.73)
+		(diameter 0)
+		(color 0 0 0 0)
+	)
+	(junction
 		(at 68.58 87.63)
 		(diameter 0)
@@
 	(wire
 		(pts
-			(xy 114.3 57.15) (xy 114.3 63.5)
-		)
-		(stroke
-			(width 0)
-			(type default)
-		)
-	)
-	(wire
-		(pts
 			(xy 107.95 118.11) (xy 107.95 82.55)
 		)
@@
 	(wire
 		(pts
-			(xy 25.4 57.15) (xy 114.3 57.15)
-		)
-		(stroke
-			(width 0)
-			(type default)
-		)
-	)
-	(wire
-		(pts
 			(xy 92.71 91.44) (xy 92.71 90.17)
 		)
@@
 	(wire
 		(pts
+			(xy 123.19 59.69) (xy 114.3 59.69)
+		)
+		(stroke
+			(width 0)
+			(type default)
+		)
+	)
+	(wire
+		(pts
 			(xy 62.23 69.85) (xy 62.23 116.84)
 		)
@@
 	(wire
 		(pts
-			(xy 25.4 71.12) (xy 25.4 57.15)
-		)
-		(stroke
-			(width 0)
-			(type default)
-		)
-	)
-	(wire
-		(pts
 			(xy 41.91 73.66) (xy 41.91 76.2)
 		)
@@
 	(wire
 		(pts
+			(xy 123.19 149.86) (xy 26.67 149.86)
+		)
+		(stroke
+			(width 0)
+			(type default)
+		)
+	)
+	(wire
+		(pts
 			(xy 77.47 87.63) (xy 77.47 95.25)
 		)
@@
 	(wire
 		(pts
+			(xy 114.3 59.69) (xy 114.3 63.5)
+		)
+		(stroke
+			(width 0)
+			(type default)
+		)
+	)
+	(wire
+		(pts
 			(xy 52.07 133.35) (xy 52.07 104.14)
 		)
@@
 	(wire
 		(pts
-			(xy 25.4 76.2) (xy 26.67 76.2)
-		)
-		(stroke
-			(width 0)
-			(type default)
-		)
-	)
-	(wire
-		(pts
 			(xy 85.09 82.55) (xy 85.09 116.84)
 		)
@@
 	(wire
 		(pts
+			(xy 123.19 64.77) (xy 123.19 149.86)
+		)
+		(stroke
+			(width 0)
+			(type default)
+		)
+	)
+	(wire
+		(pts
 			(xy 62.23 116.84) (xy 68.58 116.84)
+		)
+		(stroke
+			(width 0)
+			(type default)
+		)
+	)
+	(wire
+		(pts
+			(xy 26.67 149.86) (xy 26.67 125.73)
 		)
 		(stroke
@@
 	(symbol
 		(lib_id "Connector:Barrel_Jack")
-		(at 17.78 73.66 0)
+		(at 130.81 62.23 180)
 		(unit 1)
 		(exclude_from_sim no)
@@
 		(dnp no)
 		(property "Reference" "J3"
-			(at 17.78 64.77 0)
+			(at 130.81 71.12 0)
 			(effects
 				(font
@@
 		)
 		(property "Value" "Barrel_Jack"
-			(at 17.78 67.31 0)
+			(at 130.81 68.58 0)
 			(effects
 				(font
@@
 		)
 		(property "Footprint" "Connector_BarrelJack:BarrelJack_Horizontal"
-			(at 19.05 74.676 0)
+			(at 129.54 61.214 0)
 			(effects
 				(font
@@
 		)
 		(property "Datasheet" "~"
-			(at 19.05 74.676 0)
+			(at 129.54 61.214 0)
 			(effects
 				(font
@@
 		)
 		(property "Description" "DC Barrel Jack"
-			(at 17.78 73.66 0)
-			(effects
-				(font
+			(at 130.81 62.23 0)
+			(effects
+				(font
